File: hardware/0.1/stm32f103-feather.kicad_pcb (KiCad board)
At the start: 2 copper layers, 51.8 x 22.9 mm, 41 parts, among them J1 1.27_SWD, J2 USB_C_Receptacle_USB2.0, J3 JST_PH, J4 Feather, Q1 DMP2045U, SW1 SW_Push, SW2 SW_Push, U1 STM32F103C8Tx, U2 AP2112K-3.3, U3 MCP73831-2-OT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

Commit message: generated gerbers for V0.1
Other:
- board text added: "JLCJLC JLCJLC"
Changed lines of the file:
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@@
   (general
     (thickness 1.6)
-    (drawings 55)
+    (drawings 56)
     (tracks 696)
     (zones 0)
@@
     )
   )
+  (gr_text "JLCJLC\nJLCJLC" (at 160.3 99.5) (layer F.SilkS)
+    (effects (font (size 0.75 0.75) (thickness 0.15)))
+  )
   (gr_text A5 (at 158.5 109.4) (layer F.SilkS)
     (effects (font (size 0.75 0.75) (thickness 0.15)))
@@
     (effects (font (size 0.75 0.75) (thickness 0.15)) (justify mirror))
   )
-  (gr_text MISO (at 166.2 109.4) (layer B.SilkS)
+  (gr_text MISO (at 166.4 109.4) (layer B.SilkS)
     (effects (font (size 0.75 0.75) (thickness 0.15)) (justify mirror))
   )
