File: hardware/0.1/stm32f103-feather.sch (KiCad schematic (older format))
At the start: 39 parts, among them J1 1.27_SWD, J2 USB_C_Receptacle_USB2.0, J3 JST_PH, J4 Feather, Q1 DMP2045U, SW1 SW_Push, SW2 SW_Push, U1 STM32F103C8Tx, U2 AP2112K-3.3, U3 MCP73831-2-OT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

Commit message: schematic things
Parts:
- RN1: symbol josh-passive:RN -> stm32f103-feather-rescue:RN-josh-passive
Connections:
- no-connect marks 4 -> 9
Changed lines of the file:
@@
 EESchema Schematic File Version 4
-LIBS:stm32f103-feather-cache
 EELAYER 30 0
 EELAYER END
@@
 nLED_B
 $Comp
-L josh-passive:RN RN1
+L stm32f103-feather-rescue:RN-josh-passive RN1
 U 2 1 5E470D79
 P 9900 5950
@@
 $EndComp
 $Comp
-L josh-passive:RN RN1
+L stm32f103-feather-rescue:RN-josh-passive RN1
 U 3 1 5E47191D
 P 9900 6150
@@
 $EndComp
 $Comp
-L josh-passive:RN RN1
+L stm32f103-feather-rescue:RN-josh-passive RN1
 U 4 1 5E47241A
 P 8600 5950
@@
 $EndComp
 $Comp
-L josh-passive:RN RN1
+L stm32f103-feather-rescue:RN-josh-passive RN1
 U 1 1 5E4736FB
 P 9900 5750
@@
 Wire Wire Line
 	2150 5900 2450 5900
+NoConn ~ 3750 5600
+NoConn ~ 3750 5700
+NoConn ~ 2450 4300
+NoConn ~ 2450 4400
+NoConn ~ 2450 4500
 $EndSCHEMATC

Commit message: bitbang spi appears to work
Parts:
- RN1: symbol stm32f103-feather-rescue:RN-josh-passive -> josh-passive:RN
Connections:
- no-connect marks 9 -> 4
Changed lines of the file:
@@
 EESchema Schematic File Version 4
+LIBS:stm32f103-feather-cache
 EELAYER 30 0
 EELAYER END
@@
 nLED_B
 $Comp
-L stm32f103-feather-rescue:RN-josh-passive RN1
+L josh-passive:RN RN1
 U 2 1 5E470D79
 P 9900 5950
@@
 $EndComp
 $Comp
-L stm32f103-feather-rescue:RN-josh-passive RN1
+L josh-passive:RN RN1
 U 3 1 5E47191D
 P 9900 6150
@@
 $EndComp
 $Comp
-L stm32f103-feather-rescue:RN-josh-passive RN1
+L josh-passive:RN RN1
 U 4 1 5E47241A
 P 8600 5950
@@
 $EndComp
 $Comp
-L stm32f103-feather-rescue:RN-josh-passive RN1
+L josh-passive:RN RN1
 U 1 1 5E4736FB
 P 9900 5750
@@
 Wire Wire Line
 	2150 5900 2450 5900
-NoConn ~ 3750 5600
-NoConn ~ 3750 5700
-NoConn ~ 2450 4300
-NoConn ~ 2450 4400
-NoConn ~ 2450 4500
 $EndSCHEMATC
