File: hardware/0.2/stm32f103-feather.sch (KiCad schematic (older format))
At the start: 39 parts, among them J1 1.27_SWD, J2 USB_C_Receptacle_USB2.0, J3 JST_PH, J4 Feather, Q1 DMP2045U, SW1 SW_Push, SW2 SW_Push, U1 STM32F103C8Tx, U2 AP2112K-3.3, U3 MCP73831-2-OT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

Commit message: hardware
Parts:
- D1: footprint Diode_SMD:D_SOD-123F -> josh-passives-smt:D_SOD-123FL
- D4: footprint josh-led:LED_0606 -> josh-led:LED_0606_E6C0606RGBC3UDA
- RN1: symbol stm32f103-feather-rescue:RN-josh-passive -> josh-passive:RN
Changed lines of the file:
@@
 F 0 "D1" H 3350 1384 50  0000 C CNN
 F 1 "MBR120" H 3350 1475 50  0000 C CNN
-F 2 "Diode_SMD:D_SOD-123F" H 3350 1600 50  0001 C CNN
+F 2 "josh-passives-smt:D_SOD-123FL" H 3350 1600 50  0001 C CNN
 F 3 "~" H 3350 1600 50  0001 C CNN
 	1    3350 1600
@@
 F 0 "D4" H 10400 6447 50  0000 C CNN
 F 1 "LED_RGBA" H 10400 6356 50  0000 C CNN
-F 2 "josh-led:LED_0606" H 10400 5900 50  0001 C CNN
+F 2 "josh-led:LED_0606_E6C0606RGBC3UDA" H 10400 5900 50  0001 C CNN
 F 3 "~" H 10400 5900 50  0001 C CNN
 	1    10400 5950
@@
 nLED_B
 $Comp
-L stm32f103-feather-rescue:RN-josh-passive RN1
+L josh-passive:RN RN1
 U 2 1 5E470D79
 P 9900 5950
@@
 $EndComp
 $Comp
-L stm32f103-feather-rescue:RN-josh-passive RN1
+L josh-passive:RN RN1
 U 3 1 5E47191D
 P 9900 6150
@@
 $EndComp
 $Comp
-L stm32f103-feather-rescue:RN-josh-passive RN1
+L josh-passive:RN RN1
 U 4 1 5E47241A
 P 8600 5950
@@
 $EndComp
 $Comp
-L stm32f103-feather-rescue:RN-josh-passive RN1
+L josh-passive:RN RN1
 U 1 1 5E4736FB
 P 9900 5750
